File: kicad/vibamix_xiao/vibamix_xiao.kicad_pcb (KiCad board)
At the start: 4 copper layers, 67 x 27 mm, 40 parts, among them J1 SWD TagConnect, J2 SWD TagConnect, J4 Conn_01x24_MountingPin, Q1 20V 4.2A, Q2 AO3400A, T1 Tab, T2 Tab, T3 Tab, T4 Tab, U1 XIAO-nRF54l15-SMD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

Commit message: PCBA Rev A
Parts:
- removed H1, H2: M2.5 Mounting Hole, Custom_MountingHole:MountingHole_2.7mm_M2.5_Isolated
- added C12: 300pF, Capacitor_SMD:C_0402_1005Metric, B.Cu at (123.3, 98.6)
- added C13: 300pF, Capacitor_SMD:C_0402_1005Metric, B.Cu at (123.3, 96.7)
- added FID1: Fiducial, Custom_Fiducial:Fiducial_0.5mm_Mask1mm_NoCourtyard, F.Cu at (144.9, 105.4)
- added FID2: Fiducial, Custom_Fiducial:Fiducial_0.5mm_Mask1mm_NoCourtyard, F.Cu at (90.9, 105.4)
- added FID3: Fiducial, Custom_Fiducial:Fiducial_0.5mm_Mask1mm_NoCourtyard, F.Cu at (79.9, 80.4)
- added FID4: Fiducial, Custom_Fiducial:Fiducial_0.5mm_Mask1mm_NoCourtyard, B.Cu at (79.9, 80.4)
- added FID5: Fiducial, Custom_Fiducial:Fiducial_0.5mm_Mask1mm_NoCourtyard, B.Cu at (144.9, 105.4)
- added FID6: Fiducial, Custom_Fiducial:Fiducial_0.5mm_Mask1mm_NoCourtyard, B.Cu at (90.9, 105.4)
- added GRAPHIC2: Bird Logo, Custom_Graphic:BirdWithPants_Small_Right, B.Cu at (88.9, 101.9)
- added J3: Conn_01x02_MountingPin, Connector_Molex:Molex_PicoBlade_53261-0271_1x02-1MP_P1.25mm_Horizontal, B.Cu at (120.0, 91.3)
- added J5: Nordic NFC Antenna Connector, Custom_Connector_FFC-FPC:FPC-SMD_5P-P0.50_HCTL_HC-FPC-05-10-5RLTAG, B.Cu at (120.8, 97.7)
- added R2: 2.2k, Resistor_SMD:R_0402_1005Metric, B.Cu at (125.8, 104.3)
- added R4: 2.2k, Resistor_SMD:R_0402_1005Metric, B.Cu at (124.8, 104.3)
- added T5: Tab, kikit:Tab, F.Cu at (88.7, 106.4)
- added T6: Tab, kikit:Tab, F.Cu at (127.2, 106.4)
- GRAPHIC1: moved to B.Cu
- J4: footprint Custom_FFC-FPC:Hirose_FH34SRJ-24S-0.5SH_1x24-1MP_P0.50mm_Horizontal_Mirrored -> Custom_Connector_FFC-FPC:Hirose_FH34SRJ-24S-0.5SH_1x24-1MP_P0.50mm_Horizontal_Mirrored
- PART1: footprint Custom_Display:GDEY027T91-FL02 -> Custom_Display:GDEY027T91_NoSlot
- PCB1: value PCB_PN-A -> 010260011-A; moved to B.Cu
- Q1: value 20V 4.2A -> 20V 5A
- moved T4 110.9 mm to (78.9, 93.6)
- moved T3 110.4 mm to (86.9, 79.3), turned to -90 degrees
- moved GRAPHIC1 99.5 mm to (85.2, 101.9), turned to 180 degrees
- moved PCB1 95.2 mm to (79.9, 99.9), turned to 90 degrees
- moved TP2 77.4 mm to (144.4, 103.0), turned to 0 degrees
- moved TP1 77.3 mm to (143.0, 105.0), turned to 0 degrees
- moved U2 75.1 mm to (80.6, 104.0), turned to 90 degrees
- moved D7 71.2 mm to (140.0, 104.0), turned to 180 degrees
- moved C2 71.2 mm to (82.9, 104.0), turned to 90 degrees
- moved T2 69.8 mm to (140.1, 82.4), turned to -90 degrees
- moved D4 65.0 mm to (86.9, 104.0), turned to 180 degrees
- moved J2 61.7 mm to (133.4, 104.4), turned to 180 degrees
- moved U1 51.6 mm to (135.4, 92.4), turned to 0 degrees
- moved T1 49.3 mm to (145.9, 99.7), turned to 180 degrees
- moved D6 47.9 mm to (122.3, 104.0), turned to 180 degrees
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Connections:
- U1 pad 31: Net-(J3-Pin_2) -> /BATT+
- U1 pad 33: unconnected-(U1-P1.03_NFC2-Pad33) -> Net-(J5-Pin_4)
- U1 pad 34: unconnected-(U1-P1.02_NFC1-Pad34) -> Net-(J5-Pin_2)
Routing:
- net Net-(J1-~{RESET}): track 36.6 -> 58.2 mm
- net Net-(J1-SWDIO): track 36.8 -> 57.6 mm
- net Net-(J1-SWCLK): track 40.3 -> 60.6 mm
- net +3V3: track 5.47 -> 12.9 mm
- net Net-(J5-Pin_4): track 0.00 -> 3.90 mm
- net Net-(J5-Pin_2): track 0.00 -> 3.70 mm
- net /LIGHT_SENSOR_SDA: track 54.4 -> 56.9 mm, vias 1 -> 2
- net /LIGHT_SENSOR_SCL: track 53.1 -> 55.1 mm, vias 1 -> 2
- net /SPI_MOSI: track 45.7 -> 44.0 mm
- net /SPI_CLK: track 39.7 -> 38.1 mm
- net /~{SCREEN_CS}: track 37.1 -> 35.5 mm
- net /SCREEN_BUSY: track 48.4 -> 46.8 mm
- net /~{SCREEN_D/C}: track 54.0 -> 52.5 mm
- net Net-(J2-~{RESET}): track 17.8 -> 19.2 mm, vias 0 -> 2
- net /~{SCREEN_RES}: track 51.3 -> 49.9 mm
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- added copper zone on B.Cu, net /BATT+
Other:
- outline, holes or cut-outs redrawn
- board text added: "+ -"
- board text added: "BATTERY"
- board text added: "FABRICATION SPECIFIC NOTES 1. VIAS A. ALL VIAS EPOXY FILLED AND CAPPED WITH COPPER. 2. IMPEDANCE CONTROL NOT REQUIRED. 3. SOLDERMASK A. COLOR: BLACK"
- board text added: "GND"
- board text added: "NFC"
- board text added: "SAMD11"
- board text added: "VBUS"
- board text added: "ePaper"
- board text added: "nRF54"
- board text added: "vibamix"
- board text removed: "FABRICATION SPECIFIC NOTES 1. VIAS A. ALL VIAS EPOXY FILLED AND CAPPED WITH COPPER. 2. IMPEDANCE CONTROL A. ALL 0.26MM WIDE / 0.15MM SPACE TRACES ON F.CU MUST BE 50 OHMS SINGLE ENDED. COPLANAR WAVEGUIDE REFERENCED TO IN1.CU. B. SEE IMPEDANCE_CONTROL.XLSX FOR DETAILS. 3. SOLDERMASK A. COLOR: GREEN 4. HARD GOLD A. HARD GOLD PLATE EDGE CONNECTOR CONTACTS IN AREA LABELLED {dblquote}HARD GOLD PLATING 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"
