File: kicad/vibamix_xiao/vibamix_xiao.kicad_sch (KiCad schematic)
At the start: 43 parts, among them J1 SWD TagConnect, J2 SWD TagConnect, J3 Conn_01x02_Socket, J4 Conn_01x24_MountingPin, Q1 20V 4.2A, Q2 AO3400A, T1 Tab, T2 Tab, T3 Tab, T4 Tab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

Commit message: PCBA Rev A
Parts:
- removed H1, H2: M2.5 Mounting Hole, Custom_MountingHole:MountingHole_2.7mm_M2.5_Isolated, symbol Mechanical:MountingHole
- added C12, C13: 300pF, Capacitor_SMD:C_0402_1005Metric, symbol Device:C
- added FID1, FID2, FID3, FID4, FID5, FID6: Fiducial, Custom_Fiducial:Fiducial_0.5mm_Mask1mm_NoCourtyard, symbol Mechanical:Fiducial
- added GRAPHIC2: Bird Logo, Custom_Graphic:BirdWithPants_Small_Right, symbol Custom_Placeholder:Graphic
- added J5: Nordic NFC Antenna Connector, Custom_Connector_FFC-FPC:FPC-SMD_5P-P0.50_HCTL_HC-FPC-05-10-5RLTAG, symbol Connector_Generic_MountingPin:Conn_01x05_MountingPin
- added T5, T6: Tab, kikit:Tab, symbol kikit:Tab
- J3: value Conn_01x02_Socket -> Conn_01x02_MountingPin; footprint (none) -> Connector_Molex:Molex_PicoBlade_53261-0271_1x02-1MP_P1.25mm_Horizontal; symbol Connector:Conn_01x02_Socket -> Connector_Generic_MountingPin:Conn_01x02_MountingPin; MPN (none) -> 0532610271; Manufacturer (none) -> Molex
- J4: footprint Custom_FFC-FPC:Hirose_FH34SRJ-24S-0.5SH_1x24-1MP_P0.50mm_Horizontal_Mirrored -> Custom_Connector_FFC-FPC:Hirose_FH34SRJ-24S-0.5SH_1x24-1MP_P0.50mm_Horizontal_Mirrored; MPN (none) -> FH34SRJ-24S-0.5SH(50); Manufacturer (none) -> Hirose Electric Co Ltd
- PART1: footprint Custom_Display:GDEY027T91-FL02 -> Custom_Display:GDEY027T91_NoSlot
- Q1: value 20V 4.2A -> 20V 5A; symbol Device:Q_PMOS_GSD -> Transistor_FET:Q_PMOS_GSD; Manufacturer (none) -> Diodes Incorporated
- Q2: MPN (none) -> AO3400A; Manufacturer (none) -> Alpha & Omega Semiconductor Inc.
- R1: MPN (none) -> RC0402FR-07100KL
- R2, R4: footprint (none) -> Resistor_SMD:R_0402_1005Metric; MPN (none) -> RC0402FR-072K2L
- U2: MPN (none) -> LTR-329ALS-01; Manufacturer (none) -> Lite-On Inc.
Connections:
- net GND: now also J3.MP (MountPin), C12.2, C13.2, J5.MP (MountPin)
- net BATT+: now reaches J3.2 (Pin_2), U1.31 (BAT)
- net at U1.33 (P1.03_NFC2): now also C13.1, J5.4 (Pin_4)
- net at U1.34 (P1.02_NFC1): now also C12.1, J5.2 (Pin_2)
- no-connect marks 11 -> 20
Other:
- moved on the sheet: PCB1
